File: interface.kicad_sch (KiCad schematic)
At the start: 27 parts

Commit message: finished schematics
Parts:
- added R57: 3k3, Resistor_SMD:R_0603_1608Metric, symbol Device:R
- added R66: 1k, Resistor_SMD:R_0603_1608Metric, symbol Device:R
- gave numbers to parts that had none: 27
Connections:
- net ENABLE-: now also R66.1
- net TEMP_MOT: now also R57.1
- new net PWM_BREAK: R66.2
- new net TEMP_MOT_IN: R57.2
Other:
- company: (none) -> UNIMOC universal motor controller
- title: (none) -> (BCC) Battery Case Controller

Commit message: Placing first round finished
Parts:
- renumbered C72 to C75, C65 to C76, C66 to C77, C67 to C78, C69 to C79, C70 to C80, C68 to C81, C71 to C82, D30 to D40, R49 to R65, R50 to R66, R51 to R67, R52 to R68, R61 to R69, R53 to R70, R54 to R71, R55 to R72, R56 to R73, R67 to R74, R57 to R75, R64 to R76, R58 to R77, R65 to R78, R66 to R79, R62 to R80, R59 to R81, R60 to R82, R63 to R83, U32 to U42

Commit message: just the silk open
Parts:
- renumbered C75 to C81, C76 to C82, C77 to C83, C78 to C84, C79 to C85, C80 to C86, C81 to C87, C82 to C88, R65 to R68, R66 to R69, R67 to R70, R68 to R71, R69 to R72, R70 to R73, R71 to R74, R72 to R75, R73 to R76, R74 to R77, R75 to R78, R76 to R79, R77 to R80, R78 to R81, R79 to R82, R80 to R83, R81 to R84, R82 to R85, R83 to R86
Changed lines of the file:
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@@
   (symbol (lib_id "Device:C") (at 99.06 87.63 0) (unit 1)
     (in_bom yes) (on_board yes)
-    (property "Reference" "C77" (id 0) (at 97.79 86.36 90)
+    (property "Reference" "C83" (id 0) (at 97.79 86.36 90)
       (effects (font (size 1.27 1.27)) (justify left))
     )
@@
   (symbol (lib_id "Device:C") (at 106.68 87.63 0) (unit 1)
     (in_bom yes) (on_board yes)
-    (property "Reference" "C78" (id 0) (at 105.41 86.36 90)
+    (property "Reference" "C84" (id 0) (at 105.41 86.36 90)
       (effects (font (size 1.27 1.27)) (justify left))
     )
@@
   (symbol (lib_id "Device:C") (at 121.92 87.63 0) (unit 1)
     (in_bom yes) (on_board yes)
-    (property "Reference" "C80" (id 0) (at 120.65 86.36 90)
+    (property "Reference" "C86" (id 0) (at 120.65 86.36 90)
       (effects (font (size 1.27 1.27)) (justify left))
     )
@@
   (symbol (lib_id "Device:R") (at 64.77 66.04 270) (unit 1)
     (in_bom yes) (on_board yes)
-    (property "Reference" "R73" (id 0) (at 63.5 66.04 90)
+    (property "Reference" "R76" (id 0) (at 63.5 66.04 90)
       (effects (font (size 1.27 1.27)) (justify left))
     )
@@
   (symbol (lib_id "Device:R") (at 64.77 59.69 270) (unit 1)
     (in_bom yes) (on_board yes)
-    (property "Reference" "R72" (id 0) (at 63.5 59.69 90)
+    (property "Reference" "R75" (id 0) (at 63.5 59.69 90)
       (effects (font (size 1.27 1.27)) (justify left))
     )
@@
   (symbol (lib_id "Device:R") (at 64.77 53.34 270) (unit 1)
     (in_bom yes) (on_board yes)
-    (property "Reference" "R71" (id 0) (at 63.5 53.34 90)
+    (property "Reference" "R74" (id 0) (at 63.5 53.34 90)
       (effects (font (size 1.27 1.27)) (justify left))
     )
@@
   (symbol (lib_id "Device:R") (at 44.45 38.1 0) (unit 1)
     (in_bom yes) (on_board yes)
-    (property "Reference" "R66" (id 0) (at 44.45 39.37 90)
+    (property "Reference" "R69" (id 0) (at 44.45 39.37 90)
       (effects (font (size 1.27 1.27)) (justify left))
     )
@@
   (symbol (lib_id "Device:R") (at 49.53 38.1 0) (unit 1)
     (in_bom yes) (on_board yes)
-    (property "Reference" "R67" (id 0) (at 49.53 39.37 90)
+    (property "Reference" "R70" (id 0) (at 49.53 39.37 90)
       (effects (font (size 1.27 1.27)) (justify left))
     )
@@
   (symbol (lib_id "Device:R") (at 54.61 38.1 0) (unit 1)
     (in_bom yes) (on_board yes)
-    (property "Reference" "R68" (id 0) (at 54.61 39.37 90)
+    (property "Reference" "R71" (id 0) (at 54.61 39.37 90)
       (effects (font (size 1.27 1.27)) (justify left))
     )
@@
   (symbol (lib_id "Device:R") (at 39.37 38.1 0) (unit 1)
     (in_bom yes) (on_board yes)
-    (property "Reference" "R65" (id 0) (at 39.37 39.37 90)
+    (property "Reference" "R68" (id 0) (at 39.37 39.37 90)
       (effects (font (size 1.27 1.27)) (justify left))
     )
@@
   (symbol (lib_id "Device:C") (at 114.3 87.63 0) (unit 1)
     (in_bom yes) (on_board yes)
-    (property "Reference" "C79" (id 0) (at 113.03 86.36 90)
+    (property "Reference" "C85" (id 0) (at 113.03 86.36 90)
       (effects (font (size 1.27 1.27)) (justify left))
     )
@@
   (symbol (lib_id "Device:R") (at 64.77 46.99 270) (unit 1)
     (in_bom yes) (on_board yes)
-    (property "Reference" "R70" (id 0) (at 63.5 46.99 90)
+    (property "Reference" "R73" (id 0) (at 63.5 46.99 90)
       (effects (font (size 1.27 1.27)) (justify left))
     )
@@
   (symbol (lib_id "Device:R") (at 82.55 38.1 0) (unit 1)
     (in_bom yes) (on_board yes)
-    (property "Reference" "R69" (id 0) (at 82.55 39.37 90)
+    (property "Reference" "R72" (id 0) (at 82.55 39.37 90)
       (effects (font (size 1.27 1.27)) (justify left))
     )
@@
   (symbol (lib_id "Device:C") (at 82.55 87.63 0) (mirror y) (unit 1)
     (in_bom yes) (on_board yes)
-    (property "Reference" "C76" (id 0) (at 83.82 86.36 90)
+    (property "Reference" "C82" (id 0) (at 83.82 86.36 90)
       (effects (font (size 1.27 1.27)) (justify left))
     )
@@
   (symbol (lib_id "Device:C") (at 124.46 171.45 0) (unit 1)
     (in_bom yes) (on_board yes)
-    (property "Reference" "C82" (id 0) (at 123.19 170.18 90)
+    (property "Reference" "C88" (id 0) (at 123.19 170.18 90)
       (effects (font (size 1.27 1.27)) (justify left))
     )
@@
   (symbol (lib_id "Device:R") (at 90.17 149.86 270) (unit 1)
     (in_bom yes) (on_board yes)
-    (property "Reference" "R80" (id 0) (at 88.9 149.86 90)
+    (property "Reference" "R83" (id 0) (at 88.9 149.86 90)
       (effects (font (size 1.27 1.27)) (justify left))
     )
@@
   (symbol (lib_id "Device:R") (at 64.77 140.97 0) (unit 1)
     (in_bom yes) (on_board yes)
-    (property "Reference" "R77" (id 0) (at 64.77 142.24 90)
+    (property "Reference" "R80" (id 0) (at 64.77 142.24 90)
       (effects (font (size 1.27 1.27)) (justify left))
     )
@@
   (symbol (lib_id "Device:R") (at 64.77 156.21 270) (unit 1)
     (in_bom yes) (on_board yes)
-    (property "Reference" "R81" (id 0) (at 63.5 156.21 90)
+    (property "Reference" "R84" (id 0) (at 63.5 156.21 90)
       (effects (font (size 1.27 1.27)) (justify left))
     )
@@
   (symbol (lib_id "Device:R") (at 64.77 162.56 270) (unit 1)
     (in_bom yes) (on_board yes)
-    (property "Reference" "R82" (id 0) (at 63.5 162.56 90)
+    (property "Reference" "R85" (id 0) (at 63.5 162.56 90)
       (effects (font (size 1.27 1.27)) (justify left))
     )
@@
   (symbol (lib_id "Device:R") (at 97.79 171.45 180) (unit 1)
     (in_bom yes) (on_board yes)
-    (property "Reference" "R83" (id 0) (at 97.79 170.18 90)
+    (property "Reference" "R86" (id 0) (at 97.79 170.18 90)
       (effects (font (size 1.27 1.27)) (justify left))
     )
@@
   (symbol (lib_id "Device:C") (at 107.95 171.45 0) (unit 1)
     (in_bom yes) (on_board yes)
-    (property "Reference" "C81" (id 0) (at 106.68 170.18 90)
+    (property "Reference" "C87" (id 0) (at 106.68 170.18 90)
       (effects (font (size 1.27 1.27)) (justify left))
     )
@@
   (symbol (lib_id "Device:C") (at 246.38 81.28 0) (mirror y) (unit 1)
     (in_bom yes) (on_board yes)
-    (property "Reference" "C75" (id 0) (at 247.65 80.01 90)
+    (property "Reference" "C81" (id 0) (at 247.65 80.01 90)
       (effects (font (size 1.27 1.27)) (justify left))
     )
@@
   (symbol (lib_id "Device:R") (at 208.28 143.51 90) (unit 1)
     (in_bom yes) (on_board yes)
-    (property "Reference" "R78" (id 0) (at 209.55 143.51 90)
+    (property "Reference" "R81" (id 0) (at 209.55 143.51 90)
       (effects (font (size 1.27 1.27)) (justify left))
     )
@@
   (symbol (lib_id "Device:R") (at 259.08 66.04 270) (unit 1)
     (in_bom yes) (on_board yes)
-    (property "Reference" "R74" (id 0) (at 257.81 66.04 90)
+    (property "Reference" "R77" (id 0) (at 257.81 66.04 90)
       (effects (font (size 1.27 1.27)) (justify left))
     )
@@
   (symbol (lib_id "Device:R") (at 190.5 87.63 270) (unit 1)
     (in_bom yes) (on_board yes)
-    (property "Reference" "R76" (id 0) (at 190.5 87.63 90))
+    (property "Reference" "R79" (id 0) (at 190.5 87.63 90))
     (property "Value" "1R" (id 1) (at 195.58 86.36 90))
     (property "Footprint" "Resistor_SMD:R_0603_1608Metric" (id 2) (at 190.5 85.852 90)
@@
   (symbol (lib_id "Device:R") (at 64.77 72.39 270) (unit 1)
     (in_bom yes) (on_board yes)
-    (property "Reference" "R75" (id 0) (at 63.5 72.39 90)
+    (property "Reference" "R78" (id 0) (at 63.5 72.39 90)
       (effects (font (size 1.27 1.27)) (justify left))
     )
@@
   (symbol (lib_id "Device:R") (at 226.06 146.05 90) (unit 1)
     (in_bom yes) (on_board yes)
-    (property "Reference" "R79" (id 0) (at 227.33 146.05 90)
-      (effects (font (size 1.27 1.27)) (justify left))
-    )
+    (property "Reference" "R82" (id 0) (at 227.33 146.05 90)
+      (effects (font (size 1.27 1.27)) (justify left))
+    )
